Commit message: standup/model: real K1 actuator spec — freq-based gains + true torque limits
Root cause of the 6-run plateau (from Booster's own K1 Isaac config,
booster_train assets/robots/{booster,actuator}.py): our model was wrong on
BOTH gains and torque limits vs the real K1.

Torque limits (URDF effort + MJCF forcerange), per leg joint — were starving
the sim robot to ~1/3-1/2 of reality:
  knee 40->112, hip_pitch 30->68, hip_roll 35->76, hip_yaw 20->38.3,
  ankle_pitch/roll 20->38.3  (arms 14, head 6 unchanged). Shared-model fix —
  these are the REAL K1 limits, so it raises fidelity for all skills.

Gains: K1 uses frequency-based per-joint PD, kp=armature·(2π·f_n)²,
kd=2·ζ·armature·(2π·f_n), f_n=4 Hz, ζ=1.5 (hip/ankle)/1.0 (knee). Computed
from our (K1-accurate) armatures this gives kp hip30/knee60/ankle36 — NOT the
flat kp=40 (runs #1-5, too soft on knee) nor T1's kp=200 (run #6, ~3-7x too
stiff AND still torque-capped). Standup overrides _build_per_joint_gains for
legs only; arms/head keep config gains. Run #7.

Co-Authored-By: Claude Opus 4.8 <noreply@anthropic.com>

File: models/robot/K1/K1_22dof.urdf (robot description, URDF)
Before this commit: robot K1, 23 links, 22 joints
Joints:
- joint Left_Ankle_Pitch: limit lower=-0.87 upper=0.345 effort=20 velocity=18.1 -> lower=-0.87 upper=0.345 effort=38.3 velocity=18.1
- joint Left_Ankle_Roll: limit lower=-0.345 upper=0.345 effort=20 velocity=18.1 -> lower=-0.345 upper=0.345 effort=38.3 velocity=18.1
- joint Left_Hip_Pitch: limit lower=-3.0 upper=2.21 effort=30 velocity=7.1 -> lower=-3.0 upper=2.21 effort=68.0 velocity=7.1
- joint Left_Hip_Roll: limit lower=-0.4 upper=1.57 effort=35 velocity=12.9 -> lower=-0.4 upper=1.57 effort=76.0 velocity=12.9
- joint Left_Hip_Yaw: limit lower=-1. upper=1. effort=20 velocity=18.1 -> lower=-1. upper=1. effort=38.3 velocity=18.1
- joint Left_Knee_Pitch: limit lower=0. upper=2.23 effort=40 velocity=12.5 -> lower=0. upper=2.23 effort=112.0 velocity=12.5
- joint Right_Ankle_Pitch: limit lower=-0.87 upper=0.345 effort=20 velocity=18.1 -> lower=-0.87 upper=0.345 effort=38.3 velocity=18.1
- joint Right_Ankle_Roll: limit lower=-0.345 upper=0.345 effort=20 velocity=18.1 -> lower=-0.345 upper=0.345 effort=38.3 velocity=18.1
- joint Right_Hip_Pitch: limit lower=-3.0 upper=2.21 effort=30 velocity=7.1 -> lower=-3.0 upper=2.21 effort=68.0 velocity=7.1
- joint Right_Hip_Roll: limit lower=-1.57 upper=0.4 effort=35 velocity=12.9 -> lower=-1.57 upper=0.4 effort=76.0 velocity=12.9
- joint Right_Hip_Yaw: limit lower=-1. upper=1. effort=20 velocity=18.1 -> lower=-1. upper=1. effort=38.3 velocity=18.1
- joint Right_Knee_Pitch: limit lower=0. upper=2.23 effort=40 velocity=12.5 -> lower=0. upper=2.23 effort=112.0 velocity=12.5

Commit message: model: box foot colliders — fixes broken Genesis foot-ground contact
ROOT CAUSE of the standup plateau (7 runs). The K1 URDF used full-MESH foot
collision; in Genesis this gave broken/penetrating, intermittent foot contact
(feet sink through the floor; contact force flaky), so the robot never had
stable support — it always tipped/collapsed, no matter the gains/torque/reward.

Diagnostic: dropping the robot (PD-hold default pose) onto the ground —
  * mesh collider  -> collapses 0.55 -> 0.06 m in ~1.6 s (tips, bad contact)
  * box collider   -> stands STABLE at 0.539 m, foot contact ~193 N (= body
    weight), rock-steady indefinitely.

Replace the foot <collision> mesh with a box matching the MJCF collider
(size 0.18x0.07x0.036 m, origin 0.026 0 -0.02) for both feet. MJCF already used
this box for eval; now Genesis training matches it (also closes the sim2sim gap
CLAUDE.md flagged). Fixes contact for all skills (walk too).

Co-Authored-By: Claude Opus 4.8 <noreply@anthropic.com>

File: models/robot/K1/K1_22dof.urdf (robot description, URDF)
Before this commit: robot K1, 23 links, 22 joints
Links:
- link left_foot_link: geometry collision box size=0.18 0.07 0.036; visual mesh filename=meshes/Left_Foot.STL
- link right_foot_link: geometry collision box size=0.18 0.07 0.036; visual mesh filename=meshes/Right_Foot.STL
